Commit message: Make the apartment a night scene and give the robot a headlight
The world now has a dark sky, low ambient light and dim bluish moonlight
in place of the sun, matching the night thermal scene. The sphere carries
a white LED spotlight on its core, just under the RGB camera, so it tips
with the cameras and lights what they see inside the voids (assumed: about
a 1 W LED with a 50 deg beam, values in params.xacro).

Also fix the RGB camera noise: Gazebo reads the noise type from a <type>
element, not an attribute, so the noise was being ignored.

Co-Authored-By: Claude Opus 5.5 <noreply@anthropic.com>

File: src/sphere_scout_description/urdf/params.xacro (robot description, xacro)
@@ -58,4 +58,10 @@
   <xacro:property name="rgb_height" value="240"/>
   <xacro:property name="rgb_rate" value="15"/>
+  <!-- white LED headlight for the RGB camera at night (assumed: about a 1 W LED with a 50 deg
+       beam), just under the camera -->
+  <xacro:property name="headlight_xyz" value="0.031 0 0.004"/>
+  <xacro:property name="headlight_range" value="8"/>
+  <xacro:property name="headlight_inner" value="0.5"/>          <!-- rad, full-brightness cone -->
+  <xacro:property name="headlight_outer" value="0.9"/>          <!-- rad, edge of the beam -->
   <xacro:property name="imu_xyz" value="0 -0.025 -0.0195"/>
   <xacro:property name="imu_rpy" value="0 0 0"/>

File: src/sphere_scout_description/urdf/sphere.urdf.xacro (robot description, xacro)
@@ -181,6 +181,27 @@
     </sensor>
   </gazebo>
+  <!-- LED headlight on the core, so it tips with the cameras -->
+  <gazebo reference="base_link">
+    <light name="headlight" type="spot">
+      <pose>${headlight_xyz} 0 0 0</pose>
+      <direction>1 0 0</direction>
+      <diffuse>1.0 0.96 0.88 1</diffuse>
+      <specular>0.3 0.3 0.3 1</specular>
+      <attenuation>
+        <range>${headlight_range}</range>
+        <constant>0.3</constant>
+        <linear>0.12</linear>
+        <quadratic>0.04</quadratic>
+      </attenuation>
+      <spot>
+        <inner_angle>${headlight_inner}</inner_angle>
+        <outer_angle>${headlight_outer}</outer_angle>
+        <falloff>1.0</falloff>
+      </spot>
+      <cast_shadows>false</cast_shadows>
+    </light>
+  </gazebo>
   <!-- RGB feed. The OV2640 gives JPEG; in simulation gazebo_world.launch.py compresses this raw
-       image to /camera/image_raw/compressed the same way. Dark inside voids: it has no light. -->
+       image to /camera/image_raw/compressed the same way. At night it sees by the headlight. -->
   <gazebo reference="camera_link">
     <sensor name="rgb_camera" type="camera">
@@ -193,5 +214,5 @@
         <image><width>${rgb_width}</width><height>${rgb_height}</height><format>R8G8B8</format></image>
         <clip><near>0.01</near><far>50</far></clip>
-        <noise type="gaussian"><mean>0</mean><stddev>0.007</stddev></noise>
+        <noise><type>gaussian</type><mean>0</mean><stddev>0.007</stddev></noise>
       </camera>
     </sensor>
